Commit message: Base urdf with convert pose fix Added new URDF set file (as a fix for solidworks to URDF exporter) Convert position conversion fixed for inertia and relative positioning

File: urdf-sdf/URDF_Bodies2.SLDASM/urdf/URDF_Bodies2.SLDASM.urdf (robot description, URDF)
Before this commit: robot URDF_Bodies.2, 5 links, 4 joints
Links:
- link LW_Flap: mass 0.155627268196262 -> 0; geometry collision mesh filename=package://URDF_Bodies2.SLDASM/meshes/LW_Flap.STL; visual mesh filename=package://URDF_Bodies2.SLDASM/meshes/LW_Flap.STL
- link LW_Pitch: mass 2.36285860241809 -> 2.3629; geometry collision mesh filename=package://URDF_Bodies2.SLDASM/meshes/LW_Pitch.STL; visual mesh filename=package://URDF_Bodies2.SLDASM/meshes/LW_Pitch.STL
- link RW_Flap: mass 0.155627268196262 -> 0.15563; geometry collision mesh filename=package://URDF_Bodies2.SLDASM/meshes/RW_Flap.STL; visual mesh filename=package://URDF_Bodies2.SLDASM/meshes/RW_Flap.STL
- link RW_Pitch: mass 2.36285860241809 -> 2.3629; geometry collision mesh filename=package://URDF_Bodies2.SLDASM/meshes/RW_Pitch.STL; visual mesh filename=package://URDF_Bodies2.SLDASM/meshes/RW_Pitch.STL
- link base_link: mass 3.75126000883085 -> 3.7513; geometry collision mesh filename=package://URDF_Bodies2.SLDASM/meshes/base_link.STL; visual mesh filename=package://URDF_Bodies2.SLDASM/meshes/base_link.STL
Joints:
- removed joint LW_Flap
- removed joint LW_Pitch
- removed joint RW_Flap
- removed joint RW_Pitch
- added joint LW_J_Flap: type revolute, parent base_link, child LW_Flap, origin xyz=-0.12329 0 0 rpy=0 0 0, axis 0 -1 0, limit lower=0 upper=0 effort=0 velocity=0
- added joint LW_J_Pitch: type revolute, parent LW_Flap, child LW_Pitch, origin xyz=-0.09 0.04 0 rpy=0 0 0, axis 1 0 0, limit lower=0 upper=0 effort=0 velocity=0
- added joint RW_J_Flap: type revolute, parent base_link, child RW_Flap, origin xyz=0.12329 0 0 rpy=0 0 0, axis 0 -1 0, limit lower=0 upper=0 effort=0 velocity=0
- added joint RW_J_Pitch: type revolute, parent RW_Flap, child RW_Pitch, origin xyz=0.09 0.04 0 rpy=0 0 0, axis -1 0 0, limit lower=0 upper=0 effort=0 velocity=0
